File: Hardware/TFTBR.brd (EAGLE design)
At the start: 40 x 27 mm, 6 parts, among them IC1 74HC2G125, J1 SPI-LCD

Commit message: Minor updates to boards.
Parts:
- renumbered FID3 to FID2
Other:
- board text added: "TFTBR v1.0 Dimensions (mm)"
Changed lines of the file:
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@@
 <setting verticaltext="up"/>
 </settings>
-<grid distance="0.5" unitdist="mm" unit="mm" style="dots" multiple="1" display="yes" altdistance="0.001" altunitdist="inch" altunit="inch"/>
+<grid distance="1" unitdist="mm" unit="mm" style="dots" multiple="1" display="no" altdistance="0.001" altunitdist="inch" altunit="inch"/>
 <layers>
 <layer number="1" name="Top" color="59" fill="1" visible="yes" active="yes"/>
@@
 <layer number="37" name="tTest" color="7" fill="1" visible="no" active="yes"/>
 <layer number="38" name="bTest" color="7" fill="1" visible="no" active="yes"/>
-<layer number="39" name="tKeepout" color="4" fill="11" visible="yes" active="yes"/>
-<layer number="40" name="bKeepout" color="1" fill="11" visible="yes" active="yes"/>
-<layer number="41" name="tRestrict" color="4" fill="10" visible="yes" active="yes"/>
-<layer number="42" name="bRestrict" color="1" fill="10" visible="yes" active="yes"/>
+<layer number="39" name="tKeepout" color="4" fill="11" visible="no" active="yes"/>
+<layer number="40" name="bKeepout" color="1" fill="11" visible="no" active="yes"/>
+<layer number="41" name="tRestrict" color="4" fill="10" visible="no" active="yes"/>
+<layer number="42" name="bRestrict" color="1" fill="10" visible="no" active="yes"/>
 <layer number="43" name="vRestrict" color="2" fill="10" visible="no" active="yes"/>
 <layer number="44" name="Drills" color="7" fill="1" visible="no" active="yes"/>
@@
 </layers>
 <board>
-<fusionsync huburn="a.cGVyc29uYWw6dWUyZDliZmNi" projecturn="a.cGVyc29uYWw6dWUyZDliZmNiIzIwMTkwMzE1MTgyMjY5OTA2" f3durn="urn:adsk.wipprod:dm.lineage:0O-6M3RtRAKioLKEgaY_rA" pcbguid="" lastpulledtime="" lastsyncedchangeguid="42844e33-5a07-b25f-797f-d099163c2932" latestrevisionid="753c5c97-072d-40d8-b907-e1d94003c49d" lastsyncedrevisionid="753c5c97-072d-40d8-b907-e1d94003c49d" lastboardhashguid="320cd19c-a01c-2bd7-620d-10707dd9e3e8" lastpushedtime="2021-07-28T00:02:37Z" linktopcb3d="true"/>
+<fusionsync huburn="a.cGVyc29uYWw6dWUyZDliZmNi" projecturn="a.cGVyc29uYWw6dWUyZDliZmNiIzIwMTkwMzE1MTgyMjY5OTA2" f3durn="urn:adsk.wipprod:dm.lineage:ikRCzpTmRbyiFlvb3Ca_fA" pcbguid="82e6c54f-4b90-48f7-afd2-29d3e54a4c2a" lastpulledtime="" lastsyncedchangeguid="42844e33-5a07-b25f-797f-d099163c2932" latestrevisionid="16e929dc-237a-45c1-8072-94328d340520" lastsyncedrevisionid="16e929dc-237a-45c1-8072-94328d340520" lastboardhashguid="ed26078d-4b9b-ff5a-8e6c-eb0bae4e0ed8" lastpushedtime="2021-07-30T01:53:12Z" linktopcb3d="true"/>
 <plain>
 <wire x1="40" y1="25" x2="38" y2="27" width="0" layer="20" curve="90"/>
@@
 <circle x="8.6" y="7.5" radius="0.05" width="0.3048" layer="21"/>
 <wire x1="9.6" y1="9" x2="9.6" y2="9.3" width="0.3048" layer="21"/>
+<dimension x1="0" y1="28" x2="3" y2="28" x3="1.5" y3="29" textsize="1.778" layer="47" dtype="horizontal" precision="0"/>
+<dimension x1="3" y1="28" x2="37" y2="28" x3="20" y3="29" textsize="1.778" layer="47" dtype="horizontal" precision="0"/>
+<dimension x1="37" y1="28" x2="40" y2="28" x3="38.5" y3="29" textsize="1.778" layer="47" dtype="horizontal" precision="0"/>
+<dimension x1="-1" y1="2" x2="-1" y2="25" x3="-2" y3="13.5" textsize="1.778" layer="47" dtype="horizontal" precision="0"/>
+<dimension x1="-1" y1="25" x2="-1" y2="27" x3="-2" y3="26" textsize="1.778" layer="47" dtype="horizontal" precision="0"/>
+<dimension x1="-5" y1="0" x2="-5" y2="27" x3="-6" y3="13.5" textsize="1.778" layer="47" dtype="horizontal" precision="0"/>
+<dimension x1="0" y1="32" x2="37" y2="32" x3="18.5" y3="33" textsize="1.778" layer="47" dtype="horizontal" precision="0"/>
+<dimension x1="0" y1="-1" x2="20" y2="-1" x3="10" y3="-3" textsize="1.778" layer="47" dtype="horizontal" precision="0"/>
+<dimension x1="20" y1="-1" x2="40" y2="-1" x3="30" y3="-3" textsize="1.778" layer="47" dtype="horizontal" precision="0"/>
+<dimension x1="41" y1="0" x2="41" y2="13.5" x3="43" y3="6.75" textsize="1.778" layer="47" dtype="horizontal" precision="1"/>
+<dimension x1="41" y1="13.5" x2="41" y2="27" x3="43" y3="20.25" textsize="1.778" layer="47" dtype="horizontal" precision="1"/>
+<dimension x1="-1" y1="2" x2="-1" y2="0" x3="-2" y3="1" textsize="1.778" layer="47" dtype="horizontal" precision="0"/>
+<text x="3" y="37" size="1.778" layer="47">TFTBR v1.0 Dimensions (mm)</text>
 </plain>
 <attributes>
@@
 <elements>
 <element name="FID1" library="SuperHouse-Symbols" library_urn="urn:adsk.eagle:library:13228893" package="FIDUCIAL-1X2.5" package3d_urn="urn:adsk.eagle:package:13228898/2" value="FIDUCIAL1X2.5" x="3" y="18.5" smashed="yes" rot="R180"/>
-<element name="FID3" library="SuperHouse-Symbols" library_urn="urn:adsk.eagle:library:13228893" package="FIDUCIAL-1X2.5" package3d_urn="urn:adsk.eagle:package:13228898/2" value="FIDUCIAL1X2.5" x="26.833" y="8.624" smashed="yes" rot="R180"/>
+<element name="FID2" library="SuperHouse-Symbols" library_urn="urn:adsk.eagle:library:13228893" package="FIDUCIAL-1X2.5" package3d_urn="urn:adsk.eagle:package:13228898/2" value="FIDUCIAL1X2.5" x="26.833" y="8.624" smashed="yes" rot="R180"/>
 <element name="J1" library="SuperHouse-Connectors" library_urn="urn:adsk.eagle:library:11765989" package="2X04-2.54-SHROUDED" package3d_urn="urn:adsk.eagle:package:30067988/3" value="SPI-LCD" x="20" y="7" smashed="yes" rot="R180">
 <attribute name="NAME" x="20" y="12.842" size="0.8128" layer="25" font="vector" rot="R180" align="bottom-center"/>
