File: Hardware/TFTBR.sch (EAGLE design)
At the start: 6 parts, among them IC1 74HC2G125, J1 SPI-LCD

Commit message: Minor updates to boards.
Parts:
- removed FID3: FIDUCIAL1X2.5, SuperHouse-Symbols:FIDUCIAL1X2.5
- added FID2: FIDUCIAL1X2.5, SuperHouse-Symbols:FIDUCIAL1X2.5
Changed lines of the file:
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@@
 <drawing>
 <settings>
-<setting alwaysvectorfont="no"/>
+<setting alwaysvectorfont="yes"/>
 <setting keepoldvectorfont="yes"/>
 <setting verticaltext="up"/>
@@
 <parts>
 <part name="FID1" library="SuperHouse-Symbols" library_urn="urn:adsk.eagle:library:13228893" deviceset="FIDUCIAL" device="1X2.5" package3d_urn="urn:adsk.eagle:package:13228898/2"/>
-<part name="FID3" library="SuperHouse-Symbols" library_urn="urn:adsk.eagle:library:13228893" deviceset="FIDUCIAL" device="1X2.5" package3d_urn="urn:adsk.eagle:package:13228898/2"/>
+<part name="FID2" library="SuperHouse-Symbols" library_urn="urn:adsk.eagle:library:13228893" deviceset="FIDUCIAL" device="1X2.5" package3d_urn="urn:adsk.eagle:package:13228898/2"/>
 <part name="J1" library="SuperHouse-Connectors" library_urn="urn:adsk.eagle:library:11765989" deviceset="M02X4" device="-SHROUD" package3d_urn="urn:adsk.eagle:package:30067988/3" value="SPI-LCD"/>
 <part name="P+20" library="SuperHouse-SupplySymbols" library_urn="urn:adsk.eagle:library:11790503" deviceset="3.3V" device=""/>
@@
 </plain>
 <instances>
-<instance part="FID1" gate="G$1" x="106.68" y="7.62" smashed="yes"/>
-<instance part="FID3" gate="G$1" x="101.6" y="7.62" smashed="yes"/>
+<instance part="FID1" gate="G$1" x="106.68" y="10.16" smashed="yes"/>
+<instance part="FID2" gate="G$1" x="101.6" y="10.16" smashed="yes"/>
 <instance part="J1" gate="G$1" x="66.04" y="116.84" smashed="yes">
 <attribute name="VALUE" x="66.04" y="104.14" size="1.778" layer="96" align="bottom-center"/>
