File: Hardware/URC-ESP32.brd (EAGLE design)
At the start: 120 x 54 mm, 95 parts, among them IC1 MCP9808-MSOP8, IC2 ESPWROOM32, IC3 LM358D, IC4 W5500-LQFP, IC5 CP2102N-A01-GQFN24, J1 SPI-LCD, J10 microSD, J11 IO, J2 I2CBR, J3 USB-C-16P-16P, J4 DC IN, J6 PWR_LED, Q1 FDN340P, Q2 MMDT3904, U1 HY931147C-RJ45

Commit message: Fixed pin allocation notes and labels in schematic. Renamed mechanical PDF to clarify its purpose. Generated schematic PDF.
Connections:
- net IO27_T7 renamed IO27
Changed lines of the file:
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@@
 <wire x1="66" y1="3" x2="64.27" y2="4.73" width="0.254" layer="2"/>
 </signal>
-<signal name="IO27_T7">
+<signal name="IO27">
 <contactref element="IC2" pad="12"/>
 </signal>

Commit message: Minor updates to boards.
Parts:
- LED1: value YELLOW -> GREEN
- R12, R13: value 1K -> 470R
- R27, R28: value 22K -> 10K
