File: Hardware/URC-PASSTHROUGH.brd (EAGLE design)
At the start: 48 x 54 mm, 7 parts, among them J1 RJ45-X1-METAL, J2 RJ45-X1-METAL

Commit message: Schematic progress for passthrough edition.
Connections:
- removed net V+: U$1.A4, U$1.A9, U$1.B4, U$1.B9, U$2.A4, U$2.A9, U$2.B4, U$2.B9
- new net N$10: U$1.A2, U$2.A2
- new net N$11: U$1.A3, U$2.A3
- new net N$12: U$1.A4, U$2.A4
- new net N$13: U$1.A5, U$2.A5
- new net N$14: U$1.A6, U$2.A6
- new net N$15: U$1.A7, U$2.A7
- new net N$16: U$1.A8, U$2.A8
- new net N$17: U$1.A9, U$2.A9
- new net N$18: U$1.A10, U$2.A10
- new net N$19: U$1.A11, U$2.A11
- new net N$20: U$1.A12, U$2.A12
- new net N$21: U$1.B12, U$2.B12
- new net N$22: U$1.B11, U$2.B11
- new net N$23: U$1.B10, U$2.B10
- new net N$24: U$1.B9, U$2.B9
- new net N$25: U$1.B8, U$2.B8
- new net N$26: U$1.B7, U$2.B7
- new net N$27: U$1.B6, U$2.B6
- new net N$28: U$1.B5, U$2.B5
- new net N$29: U$1.B4, U$2.B4
- new net N$30: U$1.B3, U$2.B3
- new net N$31: U$1.B2, U$2.B2
- new net N$32: U$1.B1, U$2.B1
- new net N$9: U$1.A1, U$2.A1
- net GND: no longer U$1.A1, U$1.A12, U$1.B1, U$1.B12, U$2.A1, U$2.A12, U$2.B1, U$2.B12
Routing:
- net N$8: track 0.00 -> 40.9 mm
- net N$1: track 0.00 -> 38.0 mm
- net N$6: track 0.00 -> 37.9 mm
- net N$7: track 0.00 -> 25.9 mm
- net N$3: track 0.00 -> 25.0 mm
- net N$5: track 0.00 -> 23.8 mm
- net N$2: track 0.00 -> 20.9 mm
- net N$4: track 0.00 -> 18.7 mm

Commit message: Minor updates to boards.
Parts:
- removed U$2: USB-C, SuperHouse-Connectors:USB-C-U52A
- added U$3: USB-C, SuperHouse-Connectors:USB-C-U52A
Connections:
- removed net N$16: U$1.A8, U$2.A8
- removed net N$17: U$1.A9, U$2.A9
- removed net N$20: U$1.A12, U$2.A12
- removed net N$21: U$1.B12, U$2.B12
- removed net N$26: U$1.B7, U$2.B7
- removed net N$27: U$1.B6, U$2.B6
- removed net N$29: U$1.B4, U$2.B4
- removed net N$32: U$1.B1, U$2.B1
- removed net N$9: U$1.A1, U$2.A1
- net GND: now also U$1.A1, U$1.A12, U$1.B1, U$1.B12, U$3.A1, U$3.A12, U$3.B1, U$3.B12, U$3.CASE1, U$3.CASE2, U$3.CASE3, U$3.CASE4, U$3.FIX1, U$3.FIX2, U$3.FIX3, U$3.FIX4; no longer U$2.CASE1, U$2.CASE2, U$2.CASE3, U$2.CASE4, U$2.FIX1, U$2.FIX2, U$2.FIX3, U$2.FIX4
- net N$10: now also U$3.B2; no longer U$2.A2
- net N$11: now also U$3.B3; no longer U$2.A3
- net N$12: now also U$1.A8, U$3.B8; no longer U$1.A4, U$2.A4
- net N$13: now also U$3.B5; no longer U$2.A5
- net N$14: now also U$1.B6, U$3.A6, U$3.B6; no longer U$2.A6
- net N$15: now also U$1.B7, U$3.A7, U$3.B7; no longer U$2.A7
- net N$18: now also U$3.B10; no longer U$2.A10
- net N$19: now also U$3.B11; no longer U$2.A11
- net N$22: now also U$3.A11; no longer U$2.B11
- net N$23: now also U$3.A10; no longer U$2.B10
- net N$24: now also U$1.A4, U$1.A9, U$1.B4, U$3.A4, U$3.A9, U$3.B4, U$3.B9; no longer U$2.B9
- net N$25: now also U$3.A8; no longer U$2.B8
- net N$28: now also U$3.A5; no longer U$2.B5
- net N$30: now also U$3.A3; no longer U$2.B3
- net N$31: now also U$3.A2; no longer U$2.B2
Routing:
- net N$24: track 0.00 -> 33.2 mm
- net N$15: track 0.00 -> 22.4 mm
- net N$14: track 0.00 -> 19.4 mm, vias 0 -> 2
